Commit message: Track the circle in C++ and fix the Gazebo pose frame
Port the circle trajectory and control law to gtg_ros, and add a Random
trajectory button to the web UI for both backends.

The Gazebo model frame was 0.116 m ahead of the rear axle, and only the
rear axle midpoint of an Ackermann car moves as a unicycle. That left a
0.137 m steady tracking error on the circle. The model and URDF frames
are now the rear axle midpoint, and the error is 0.004 m.

Co-Authored-By: Claude Opus 5.5 <noreply@anthropic.com>
Claude-Session: https://claude.ai/code/session_01Hb6rw3t7e2BHxRwThqromV

File: gtg_ros/urdf/r2.urdf.xacro (robot description, xacro)
@@ -17,6 +17,7 @@
   <material name="tyre"><color rgba="0.2 0.2 0.2 1"/></material>
   <material name="camera"><color rgba="0.08 0.08 0.08 1"/></material>
-  <!-- Frame names follow REP-120: base_footprint on the ground below base_link, the body
-       frame. The map -> base_footprint transform is the robot pose (pose_tf_node). -->
+  <!-- Frame names follow REP-120. base_footprint is on the ground at the middle of the rear
+       axle, the same point as the Gazebo model frame, and base_link is 0.11607 m ahead of
+       it. The map -> base_footprint transform is the robot pose (pose_tf_node). -->
   <link name="base_footprint"/>
   <link name="base_link">
@@ -40,5 +41,5 @@
     <parent link="base_footprint"/>
     <child link="base_link"/>
-    <origin xyz="0 0 ${base_z}"/>
+    <origin xyz="${-wheel_base_x} 0 ${base_z}"/>
   </joint>
   <xacro:macro name="wheel" params="name parent x y">
